File: hardware/hv0a/spice-usbm.sch (EAGLE design)
At the start: 37 parts, among them J1 USB-C, J2 2X8, U1 CP2130, U10 74LVC1G17, U11 74LVC1G17, U12 74LVC1G17, U13 74LVC1G17, U14 74LVC1G17, U15 74LVC1G17, U2 74HC541, U3 74LVC1G17, U4 74LVC1G17, U5 74LVC1G17, U6 74LVC1G17, U7 74LVC1G17, U8 74LVC1G17, U9 74LVC1G17

Commit message: finished pcbs, generated gerbers
Parts:
- removed IC1: (no value), Power > LDO Voltage Regulators:MCP1700T-3302TT
- removed J1: USB-C, Connectors > USB:USB-C
- added D5: PESD5V0S1BAF, Circuit Protection > ESD Suppressors \ TVS Diodes:PESD5V0S1BAF
- added F1: (no value), Circuit Protection > Resettable Fuses - PPTC:PTC1210
- added U16: 74LVC1G17, Semiconductors > Integrated Circuits - ICs > Logic ICs > Logic Gates:74LVC1G17
- added USB1: USB_MICRO-MICRO-B-SMT, Connectors > USB:USB_MICRO-MICRO-B-SMT
- D1: value LED0603 -> SP0503BAHT; device Opto-electronics > LED Emitters:LED0603 -> Circuit Protection > ESD Suppressors \ TVS Diodes:SP0503BAHT
- D4: value SP0503BAHT -> LED0603; device Circuit Protection > ESD Suppressors \ TVS Diodes:SP0503BAHT -> Opto-electronics > LED Emitters:LED0603
- R4: device Passive Components > Resistors > Resistor Networks & Arrays:RESISTOR_4PACK -> Passive Components > Resistors > Chip Resistors:RESISTOR0603
- R7: device Passive Components > Resistors > Chip Resistors:RESISTOR0603 -> Passive Components > Resistors > Resistor Networks & Arrays:RESISTOR_4PACK
- U1: value CP2130 -> MCP1700T-3302TT; device Semiconductors > Integrated Circuits - ICs > Interface ICs > USB Interface IC:CP2130 -> Power > LDO Voltage Regulators:MCP1700T-3302TT
- U11: value 74LVC1G17 -> 74HC541; device Semiconductors > Integrated Circuits - ICs > Logic ICs > Logic Gates:74LVC1G17 -> Semiconductors > Integrated Circuits - ICs > Logic ICs > Logic Gates:74HC541
- U2: value 74HC541 -> CP2130; device Semiconductors > Integrated Circuits - ICs > Logic ICs > Logic Gates:74HC541 -> Semiconductors > Integrated Circuits - ICs > Interface ICs > USB Interface IC:CP2130
Connections:
- removed net N$15: U2.5.A, U9.1.Y
- new net OE1: U11.OE.A, U9.1.Y
- new net OE2: U10.1.Y, U11.OE.B
- net 3.3V: now also C3.P$1, R1.P$2, R2.P$1, R4.P$2, U1.VO, U13.PW.VCC, U14.PW.VCC, U2.VDD@6, U2.VIO@5, U2.VREGIN@7; no longer C1.P$1, IC1.VO, R1.P$1, R2.P$2, R7.P$2, U1.VDD@6, U1.VIO@5, U1.VREGIN@7, U10.PW.VCC, U11.PW.VCC
- net 5V: now also C1.P$1, D1.4, F1.1, U1.VI, U2.VBUS@8; no longer C3.P$1, D4.4, IC1.VI, J1.VBUS@B9,B4,A4,A9, U1.VBUS@8
- net CLKO: now also R6G$4.2, U11.4.Y; no longer R6G$4.1, U2.5.Y
- net CLKO-PB: now also U15.1.A, U2.GPIO5-!CS5!-CLKOUT@17; no longer U1.GPIO5-!CS5!-CLKOUT@17, U9.1.A
- net CS0: now also R5G$3.1, U11.2.Y; no longer R4G$3.2, U2.2.Y
- net CS0-PB: now also U2.GPIO0-!CS0@22; no longer U1.GPIO0-!CS0@22
- net CS1: now also R5G$2.1, U11.1.Y; no longer R4G$2.2, U2.3.Y
- net CS1-PB: now also U2.GPIO1-!CS1@21; no longer U1.GPIO1-!CS1@21
- net CS2: now also R5G$1.1, U11.0.Y; no longer R4G$1.2, U2.4.Y
- net CS2-PB: now also U2.GPIO2-!CS2@20; no longer U1.GPIO2-!CS2@20
- net DN: now also D1.2, U2.D-@4, USB1.D-; no longer D4.2, J1.DN@A7,B7, U1.D-@4
- net DP: now also D1.3, U2.D+@3, USB1.D+; no longer D4.3, J1.DP@A6,B6, U1.D+@3
- net EVNT: now also R6G$2.2, U13.1.A; no longer R6G$2.1, U11.1.A
- net EVNT-PB: now also U13.1.Y, U2.GPIO4-!CS4!-EVTCNTR@18; no longer U1.GPIO4-!CS4!-EVTCNTR@18, U11.1.Y
- net GND: now also D1.1, D2.CA, D5.P$2, U1.GND, U11.5.A, U11G$1.GND, U16.PW.GND, U2.GND@2, U2.GNDP, USB1.GND, USB1.SHIELD@0, USB1.SHIELD@1, USB1.SHIELD@2, USB1.SHIELD@3, USB1.SHIELD@4, USB1.SHIELD@5; no longer D3.CA, D4.1, IC1.GND, J1.GND@A12,A1,B1,B12, U1.GND@2, U1.GNDP, U11.PW.GND, U2.7.A, U2G$1.GND
- net IO6: now also R6G$1.2, U14.1.A; no longer R6G$1.1, U12.1.A
- net IO6-PB: now also U14.1.Y, U2.GPIO6-!CS6@15; no longer U1.GPIO6-!CS6@15, U12.1.Y
- net IO7: now also R7G$4.1, U11.7.Y; no longer R5G$4.1, U2.6.Y
- net IO7-PB: now also U16.1.A, U2.GPIO7-!CS7@14; no longer U1.GPIO7-!CS7@14, U13.1.A
- net MISO: now also R7G$2.1; no longer R5G$2.2
- net MISO-PB: now also U2.MISO@24; no longer U1.MISO@24
- net MOSI: now also R7G$3.1, U11.6.Y; no longer R5G$3.2, U2.0.Y
- net MOSI-PB: now also U2.MOSI@23; no longer U1.MOSI@23
- net N$1: now also U11.4.A; no longer U2.OE.B
- net N$10: now also U11.2.A, U6.1.Y; no longer U2.1.A, U5.1.Y
- net N$11: now also U11.1.A, U7.1.Y; no longer U2.2.A, U6.1.Y
- net N$12: now also U11.0.A, U8.1.Y; no longer U2.3.A, U7.1.Y
- net N$13: now also F1.2, USB1.VBUS; no longer U2.4.A, U8.1.Y
- net N$14: now also U11.7.A, U16.1.Y; no longer U13.1.Y, U2.6.A
- net N$16: now also R7G$3.2; no longer R5G$3.1
- net N$17: now also J2.5.S, R5G$1.2; no longer J2.11.S, R4G$4.1
- net N$18: now also J2.7.S, R5G$2.2; no longer J2.9.S, R4G$3.1
- net N$19: now also J2.9.S, R5G$3.2; no longer J2.7.S, R4G$2.1
- net N$2: now also D3.AN, R3.P$1; no longer D1.AN, R2.P$1
- net N$20: now also J2.11.S, R5G$4.2; no longer J2.5.S, R4G$1.1
- net N$21: now also R6G$4.1; no longer R6G$4.2
- net N$22: now also R6G$3.1; no longer R6G$3.2
- net N$23: now also R6G$2.1; no longer R6G$2.2
- net N$24: now also R6G$1.1; no longer R6G$1.2
- net N$25: now also R7G$4.2; no longer R5G$4.2
- net N$3: now also D4.AN, R4.P$1; no longer D2.AN, R3.P$1
- net N$4: now also R2.P$2, U2.!RST@9; no longer R1.P$2, U1.!RST@9
- net N$5: now also U11.3.A, U5.1.Y; no longer U14.1.Y, U2.OE.A
- net N$6: now also R7G$2.2; no longer R5G$2.1
- net N$7: now also U11.6.A; no longer U2.0.A
- net N$8: now also U2.VPP@16; no longer U1.VPP@16
- net N$9: now also D2.AN, R1.P$1; no longer D3.AN, R7.P$1
- net OEN-PB: now also U10.1.A, U2.GPIO10-!CS10!-!SUSPEND@11; no longer U1.GPIO10-!CS10!-!SUSPEND@11, U15.1.A
- net RTR: now also R6G$3.2, U12.1.A; no longer R6G$3.1, U10.1.A
- net RTR-PB: now also U12.1.Y, U2.GPIO3-!CS3!-RTR@19; no longer U1.GPIO3-!CS3!-RTR@19, U10.1.Y
- net SCK: now also R5G$4.1, U11.3.Y; no longer R4G$4.2, U2.1.Y
- net SCK-PB: now also U2.SCK@1; no longer U1.SCK@1
- net SPIACT: now also D4.CA, U2.GPIO8-!CS8!-SPIACT@13; no longer D2.CA, U1.GPIO8-!CS8!-SPIACT@13
- net SUS: now also D3.CA, U2.GPIO9-!CS9!-SUSPEND@12, U9.1.A; no longer D1.CA, U1.GPIO9-!CS9!-SUSPEND@12, U14.1.A
- net VREF: now also D5.P$1, U10.PW.VCC, U11G$1.VCC, U16.PW.VCC; no longer U13.PW.VCC, U14.PW.VCC, U2G$1.VCC
Other:
- note added: "the SPICE USB-SPI Adapter"
- note removed: "USB-SPI Adapter"
- moved on the sheet: C1, C2, C3, C4, C5, C6, C7, C8, D2, D3, J2.1, J2.10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
