File: pcb/spice-usbc.brd (EAGLE design)
At the start: 49 x 22.5 mm, 42 parts, among them J1 USB-C, J2 2X8, U1 MCP1700T-3302TT, U10 74LVC1G17, U11 74HC541, U12 74LVC1G17, U13 74LVC1G17, U14 74LVC1G17, U15 74LVC1G17, U16 74LVC1G17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

Commit message: Add USB C CC lines pull down
Parts:
- added R8, R9: 5k1, Passive Components > Resistors > Chip Resistors:0603_WAVE
Connections:
- new net N$15: J1.B5, R8.P$2
- new net N$26: J1.A5, R9.P$2
- net GND: now also R8.P$1, R9.P$1
Routing:
- net N$26: track 0.00 -> 11.6 mm, vias 0 -> 2
- net N$15: track 0.00 -> 8.55 mm, vias 0 -> 2
Other:
- board text added: "v1.0 1918"
- board text removed: "hv0a 1918"
Changed lines of the file:
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@@
 <?xml version="1.0" encoding="utf-8"?>
 <!DOCTYPE eagle SYSTEM "eagle.dtd">
-<eagle version="9.3.2">
+<eagle version="9.3.0">
 <drawing>
 <settings>
@@
 <setting verticaltext="up"/>
 </settings>
-<grid distance="0.635" unitdist="mm" unit="mm" style="lines" multiple="1" display="no" altdistance="0.0635" altunitdist="mm" altunit="mm"/>
+<grid distance="0.1" unitdist="mm" unit="mm" style="lines" multiple="1" display="no" altdistance="0.0635" altunitdist="mm" altunit="mm"/>
 <layers>
 <layer number="1" name="Top" color="4" fill="1" visible="yes" active="yes"/>
@@
 <layer number="42" name="bRestrict" color="1" fill="10" visible="yes" active="yes"/>
 <layer number="43" name="vRestrict" color="2" fill="10" visible="no" active="yes"/>
-<layer number="44" name="Drills" color="7" fill="1" visible="no" active="yes"/>
-<layer number="45" name="Holes" color="7" fill="1" visible="no" active="yes"/>
+<layer number="44" name="Drills" color="7" fill="1" visible="yes" active="yes"/>
+<layer number="45" name="Holes" color="7" fill="1" visible="yes" active="yes"/>
 <layer number="46" name="Milling" color="3" fill="1" visible="no" active="yes"/>
 <layer number="47" name="Measures" color="7" fill="1" visible="no" active="yes"/>
@@
 <wire x1="1" y1="22.5" x2="0" y2="21.5" width="0" layer="20" curve="90"/>
 <hole x="3" y="19.5" drill="3"/>
-<hole x="3" y="3" drill="3"/>
-<hole x="34" y="19.5" drill="3"/>
 <hole x="34" y="3" drill="3"/>
 <text x="19.05" y="1.905" size="1.778" layer="21" font="vector" ratio="12">the SPICE</text>
-<text x="36.83" y="1.905" size="0.8" layer="21" ratio="12">hv0a 1918</text>
+<text x="36.83" y="1.905" size="0.8" layer="21" ratio="12">v1.0 1918</text>
 </plain>
 <attributes>
@@
 </element>
 <element name="R1" library="Passive Components &gt; Resistors &gt; Chip Resistors" package="0603_WAVE" value="" x="6.858" y="3.175" smashed="yes" rot="R90">
-<attribute name="NAME" x="6.858" y="1.0795" size="0.8" layer="25" font="vector" ratio="15" rot="R180" align="center"/>
+<attribute name="NAME" x="6.7945" y="1.143" size="0.8" layer="25" font="vector" ratio="15" rot="R180" align="center"/>
 </element>
 <element name="U2" library="Semiconductors &gt; Integrated Circuits - ICs &gt; Interface ICs &gt; USB Interface IC" package="QFN24" value="CP2130" x="15" y="11.19" smashed="yes" rot="R270">
@@
 <element name="J1" library="Connectors &gt; USB" package="USB-C" value="USB-C" x="0" y="11.25" smashed="yes" rot="R270">
 <attribute name="NAME" x="8.636" y="7.44" size="0.8" layer="21" font="vector" ratio="15" rot="R90"/>
+</element>
+<element name="R8" library="Passive Components &gt; Resistors &gt; Chip Resistors" package="0603_WAVE" value="5k1" x="4.191" y="3.175" smashed="yes" rot="R90">
+<attribute name="NAME" x="4.191" y="1.143" size="0.8" layer="25" font="vector" ratio="12" align="center"/>
+</element>
+<element name="R9" library="Passive Components &gt; Resistors &gt; Chip Resistors" package="0603_WAVE" value="5k1" x="2.6035" y="3.175" smashed="yes" rot="R90">
+<attribute name="NAME" x="2.6035" y="1.143" size="0.8" layer="25" font="vector" ratio="12" rot="R180" align="center"/>
 </element>
 </elements>
@@
 <contactref element="J1" pad="B1_A12"/>
 <contactref element="J1" pad="A1_B12"/>
+<contactref element="R9" pad="P$1"/>
+<contactref element="R8" pad="P$1"/>
 </signal>
 <signal name="N$2">
@@
 <wire x1="7.216" y1="13.59" x2="6.4906" y2="13.59" width="0.3048" layer="1"/>
 </signal>
+<signal name="N$15">
+<contactref element="J1" pad="B5"/>
+<contactref element="R8" pad="P$2"/>
+<wire x1="4.191" y1="3.998" x2="4.191" y2="4.7625" width="0.2" layer="1"/>
+<wire x1="4.191" y1="4.7625" x2="4.826" y2="5.3975" width="0.2" layer="1"/>
+<via x="4.826" y="5.3975" extent="1-16" drill="0.3"/>
+<wire x1="4.826" y1="5.3975" x2="4.826" y2="9.371" width="0.2" layer="16"/>
+<wire x1="4.826" y1="9.371" x2="5.715" y2="10.26" width="0.2" layer="16"/>
+<via x="5.715" y="10.26" extent="1-16" drill="0.3"/>
+<wire x1="5.715" y1="10.26" x2="5.995" y2="9.98" width="0.2" layer="1"/>
+<wire x1="5.995" y1="9.98" x2="7.251" y2="9.98" width="0.2" layer="1"/>
+</signal>
+<signal name="N$26">
+<contactref element="J1" pad="A5"/>
+<contactref element="R9" pad="P$2"/>
+<wire x1="2.6035" y1="3.998" x2="2.6035" y2="4.8035" width="0.2" layer="1"/>
+<wire x1="2.6035" y1="4.8035" x2="3.2" y2="5.4" width="0.2" layer="1"/>
+<via x="3.2" y="5.4" extent="1-16" drill="0.3"/>
+<wire x1="3.2" y1="5.4" x2="4.2" y2="6.4" width="0.2" layer="16"/>
+<wire x1="5.7" y1="12.6" x2="4.2" y2="11.1" width="0.2" layer="16"/>
+<via x="5.7" y="12.6" extent="1-16" drill="0.3"/>
+<wire x1="5.7" y1="12.6" x2="6.1" y2="13" width="0.2" layer="1"/>
+<wire x1="6.1" y1="13" x2="7.251" y2="13" width="0.2" layer="1"/>
+<wire x1="4.2" y1="6.4" x2="4.2" y2="11.1" width="0.2" layer="16"/>
+</signal>
 </signals>

Commit message: panelize
Parts:
- removed U$3: (no value), Utility > Silkscreen:RAFAEL_SILVA_5MM_ALT_3
- added U$4: (no value), Utility > Silkscreen:RAFAEL_SILVA_10MM_ALT
- moved U$1 7.62 mm to (17.2, 1.72)
- moved U$2 1.66 mm to (31.7, 18.5)
Other:
- board text added: "C1"
- board text added: "C2"
- board text added: "C3"
- board text added: "C4"
- board text added: "C5"
- board text added: "C6"
- board text added: "C7"
- board text added: "C8"
- board text added: "D1"
- board text added: "D2"
- board text added: "D3"
- board text added: "D4"
- board text added: "D5"
- board text added: "F1"
- board text added: "J1"
- board text added: "J2"
- board text added: "R1"
- board text added: "R2"
- board text added: "R3"
- board text added: "R4"
- board text added: "R5"
- board text added: "R6"
- board text added: "R7"
- board text added: "R8"
- board text added: "R9"
- board text added: "U1"
- board text added: "U10"
- board text added: "U11"
- board text added: "U12"
- board text added: "U13"
- board text added: "U14"
- board text added: "U15"
- board text added: "U16"
- board text added: "U2"
- board text added: "U3"
- board text added: "U4"
- board text added: "U5"
- board text added: "U6"
- board text added: "U7"
- board text added: "U8"
- board text added: "U9"
- board text added: "the SPIce"
- board text removed: "the SPICE"
Changed lines of the file:
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@@
 <layer number="23" name="tOrigins" color="15" fill="1" visible="yes" active="yes"/>
 <layer number="24" name="bOrigins" color="15" fill="1" visible="yes" active="yes"/>
-<layer number="25" name="tNames" color="7" fill="1" visible="yes" active="yes"/>
+<layer number="25" name="tNames" color="7" fill="1" visible="no" active="yes"/>
 <layer number="26" name="bNames" color="7" fill="1" visible="yes" active="yes"/>
 <layer number="27" name="tValues" color="7" fill="1" visible="no" active="yes"/>
 <layer number="28" name="bValues" color="7" fill="1" visible="no" active="yes"/>
-<layer number="29" name="tStop" color="7" fill="3" visible="no" active="yes"/>
-<layer number="30" name="bStop" color="7" fill="6" visible="no" active="yes"/>
-<layer number="31" name="tCream" color="7" fill="4" visible="no" active="yes"/>
+<layer number="29" name="tStop" color="7" fill="3" visible="yes" active="yes"/>
+<layer number="30" name="bStop" color="7" fill="6" visible="yes" active="yes"/>
+<layer number="31" name="tCream" color="7" fill="4" visible="yes" active="yes"/>
 <layer number="32" name="bCream" color="7" fill="5" visible="no" active="yes"/>
 <layer number="33" name="tFinish" color="6" fill="3" visible="no" active="yes"/>
@@
 <layer number="44" name="Drills" color="7" fill="1" visible="yes" active="yes"/>
 <layer number="45" name="Holes" color="7" fill="1" visible="yes" active="yes"/>
-<layer number="46" name="Milling" color="3" fill="1" visible="no" active="yes"/>
+<layer number="46" name="Milling" color="3" fill="1" visible="yes" active="yes"/>
 <layer number="47" name="Measures" color="7" fill="1" visible="no" active="yes"/>
 <layer number="48" name="Document" color="7" fill="1" visible="no" active="yes"/>
@@
 <layer number="119" name="KAP_TEKEN" color="7" fill="1" visible="no" active="yes"/>
 <layer number="120" name="Descript" color="7" fill="1" visible="no" active="yes"/>
-<layer number="121" name="_tsilk" color="7" fill="1" visible="no" active="yes"/>
+<layer number="121" name="_tPlace" color="14" fill="1" visible="yes" active="yes"/>
 <layer number="122" name="_bsilk" color="7" fill="1" visible="no" active="yes"/>
 <layer number="123" name="tTestmark" color="7" fill="1" visible="no" active="yes"/>
 <layer number="124" name="bTestmark" color="7" fill="1" visible="no" active="yes"/>
-<layer number="125" name="_tNames" color="7" fill="1" visible="no" active="yes"/>
+<layer number="125" name="_tNames" color="14" fill="1" visible="yes" active="yes"/>
 <layer number="126" name="_bNames" color="7" fill="1" visible="no" active="yes"/>
 <layer number="127" name="_tValues" color="7" fill="1" visible="no" active="yes"/>
@@
 <hole x="3" y="19.5" drill="3"/>
 <hole x="34" y="3" drill="3"/>
-<text x="19.05" y="1.905" size="1.778" layer="21" font="vector" ratio="12">the SPICE</text>
+<text x="19.05" y="1.905" size="1.778" layer="21" font="vector" ratio="12">the SPIce</text>
 <text x="36.83" y="1.905" size="0.8" layer="21" ratio="12">v1.0 1918</text>
+<text x="10.541" y="18.796" size="0.799996875" layer="125" font="vector" ratio="15" rot="R90" align="center">C1</text>
+<text x="17.399" y="17.7165" size="0.799996875" layer="125" font="vector" ratio="15" align="center">C2</text>
+<text x="11.43" y="5.334" size="0.799996875" layer="125" font="vector" ratio="15" align="center">C3</text>
+<text x="9.8425" y="5.334" size="0.799996875" layer="125" font="vector" ratio="15" align="center">C4</text>
+<text x="19.939" y="10.287" size="0.799996875" layer="125" font="vector" ratio="15" rot="R270" align="center">C5</text>
+<text x="19.05" y="17.7165" size="0.799996875" layer="125" font="vector" ratio="15" align="center">C6</text>
+<text x="23.8125" y="6.604" size="0.799996875" layer="125" font="vector" ratio="15" align="center">C7</text>
+<text x="35.7505" y="17.2085" size="0.799996875" layer="125" font="vector" ratio="15" rot="R180" align="center">C8</text>
+<text x="8.60300625" y="12.840996875" size="0.799996875" layer="121" font="vector" ratio="15">D1</text>
+<text x="8.509" y="1.143" size="0.799996875" layer="125" font="vector" ratio="15" align="center">D2</text>
+<text x="12.2555" y="1.143" size="0.799996875" layer="125" font="vector" ratio="15" rot="R180" align="center">D3</text>
+<text x="16.1925" y="1.143" size="0.799996875" layer="125" font="vector" ratio="15" rot="R180" align="center">D4</text>
+<text x="41.275" y="19.05" size="0.799996875" layer="125" font="vector" ratio="15" rot="R180" align="center">D5</text>
+<text x="7.62" y="17.2085" size="0.799996875" layer="125" font="vector" ratio="15" rot="R180" align="center">F1</text>
+<text x="8.636" y="7.439990625" size="0.799996875" layer="121" font="vector" ratio="15" rot="R90">J1</text>
+<text x="45.8255125" y="11.697996875" size="0.799996875" layer="121" font="vector" ratio="15" rot="R270">J2</text>
+<text x="6.7945" y="1.143" size="0.799996875" layer="125" font="vector" ratio="15" rot="R180" align="center">R1</text>
+<text x="13.208" y="6.1595" size="0.799996875" layer="125" font="vector" ratio="15" align="center">R2</text>
+<text x="10.668" y="1.143" size="0.799996875" layer="125" font="vector" ratio="15" rot="R180" align="center">R3</text>
+<text x="14.605" y="1.143" size="0.799996875" layer="125" font="vector" ratio="15" rot="R180" align="center">R4</text>
+<text x="42.095496875" y="14.983509375" size="0.799996875" layer="125" font="vector" ratio="15" rot="R270" align="center">R5</text>
+<text x="42.158996875" y="9.983496875" size="0.799996875" layer="125" font="vector" ratio="15" rot="R90" align="center">R6</text>
+<text x="42.158996875" y="6.19000625" size="0.799996875" layer="125" font="vector" ratio="15" rot="R270" align="center">R7</text>
+<text x="4.191" y="1.143" size="0.799996875" layer="125" font="vector" ratio="12" align="center">R8</text>
+<text x="2.6035" y="1.143" size="0.799996875" layer="125" font="vector" ratio="12" rot="R180" align="center">R9</text>
+<text x="13.2715" y="18.4785" size="0.799996875" layer="125" font="vector" ratio="15" rot="R90" align="center">U1</text>
+<text x="18.48" y="12.146509375" size="0.799996875" layer="121" font="vector" ratio="15" rot="R90">U2</text>
+<text x="13.6525" y="14.859" size="0.799996875" layer="121" font="vector" ratio="15" rot="R180">U3</text>
+<text x="28.448" y="8.328990625" size="0.799996875" layer="121" font="vector" ratio="15" rot="R270">U4</text>
+<text x="28.3845" y="10.702009375" size="0.799996875" layer="121" font="vector" ratio="15" rot="R270">U5</text>
+<text x="20.5105" y="13.39250625" size="0.799996875" layer="121" font="vector" ratio="15" rot="R270">U6</text>
+<text x="28.3845" y="13.39250625" size="0.799996875" layer="121" font="vector" ratio="15" rot="R270">U7</text>
+<text x="20.5105" y="15.8925" size="0.799996875" layer="121" font="vector" ratio="15" rot="R270">U8</text>
+<text x="28.3845" y="15.829" size="0.799996875" layer="121" font="vector" ratio="15" rot="R270">U9</text>
+<text x="17.5895" y="6.731" size="0.799996875" layer="121" font="vector" ratio="15">U10</text>
+<text x="31.158509375" y="7.222996875" size="0.799996875" layer="125" font="vector" ratio="15" align="center">U11</text>
+<text x="17.7165" y="14.859" size="0.799996875" layer="121" font="vector" ratio="15" rot="R180">U12</text>
+<text x="23.8125" y="17.7165" size="0.799996875" layer="121" font="vector" ratio="15" rot="R180">U13</text>
+<text x="27.6225" y="17.8435" size="0.799996875" layer="121" font="vector" ratio="15" rot="R180">U14</text>
+<text x="20.5105" y="11.210009375" size="0.799996875" layer="121" font="vector" ratio="15" rot="R270">U15</text>
+<text x="20.447" y="8.646490625" size="0.799996875" layer="121" font="vector" ratio="15" rot="R270">U16</text>
 </plain>
 <attributes>
@@
 <attribute name="VALUE" x="10.16" y="23.495" size="1.27" layer="27" rot="R180"/>
 </element>
-<element name="U$1" library="Utility &gt; Silkscreen" package="DESIGNEDINPT" value="" x="20.955" y="8.3185" smashed="yes" rot="MR0"/>
-<element name="U$3" library="Utility &gt; Silkscreen" package="RAFAEL_SILVA_5MM_ALT_3" value="" x="23.495" y="13.335" smashed="yes" rot="MR0"/>
-<element name="U$2" library="Utility &gt; Silkscreen" package="OSHW-LOGO-MINI" value="" x="30.7975" y="17.145" smashed="yes"/>
+<element name="U$1" library="Utility &gt; Silkscreen" package="DESIGNEDINPT" value="" x="17.155" y="1.7185" smashed="yes" rot="MR0"/>
+<element name="U$2" library="Utility &gt; Silkscreen" package="OSHW-LOGO-MINI" value="" x="31.6975" y="18.545" smashed="yes"/>
 <element name="J1" library="Connectors &gt; USB" package="USB-C" value="USB-C" x="0" y="11.25" smashed="yes" rot="R270">
 <attribute name="NAME" x="8.636" y="7.44" size="0.8" layer="21" font="vector" ratio="15" rot="R90"/>
@@
 <attribute name="NAME" x="2.6035" y="1.143" size="0.8" layer="25" font="vector" ratio="12" rot="R180" align="center"/>
 </element>
+<element name="U$4" library="Utility &gt; Silkscreen" package="RAFAEL_SILVA_10MM_ALT" value="" x="31.6" y="6.4" smashed="yes" rot="MR0"/>
 </elements>
 <signals>
