File: pcb/spice-usbm.brd (EAGLE design)
At the start: 49 x 22.5 mm, 42 parts, among them J2 2X8, U1 MCP1700T-3302TT, U10 74LVC1G17, U11 74HC541, U12 74LVC1G17, U13 74LVC1G17, U14 74LVC1G17, U15 74LVC1G17, U16 74LVC1G17, U2 CP2130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

Commit message: panelize
Parts:
- removed U$3: (no value), Utility > Silkscreen:RAFAEL_SILVA_5MM_ALT_3
- added U$4: (no value), Utility > Silkscreen:RAFAEL_SILVA_10MM_ALT
- moved U$1 7.62 mm to (17.2, 1.72)
- moved U$2 0.30 mm to (31.1, 17.3)
Other:
- board text added: "C1"
- board text added: "C2"
- board text added: "C3"
- board text added: "C4"
- board text added: "C5"
- board text added: "C6"
- board text added: "C7"
- board text added: "C8"
- board text added: "D1"
- board text added: "D2"
- board text added: "D3"
- board text added: "D4"
- board text added: "D5"
- board text added: "F1"
- board text added: "J2"
- board text added: "R1"
- board text added: "R2"
- board text added: "R3"
- board text added: "R4"
- board text added: "R5"
- board text added: "R6"
- board text added: "R7"
- board text added: "U1"
- board text added: "U10"
- board text added: "U11"
- board text added: "U12"
- board text added: "U13"
- board text added: "U14"
- board text added: "U15"
- board text added: "U16"
- board text added: "U2"
- board text added: "U3"
- board text added: "U4"
- board text added: "U5"
- board text added: "U6"
- board text added: "U7"
- board text added: "U8"
- board text added: "U9"
- board text added: "USB1"
- board text added: "the SPIce"
- board text removed: "hv0a 1918"
- board text removed: "the SPICE"
Changed lines of the file:
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@@
 <?xml version="1.0" encoding="utf-8"?>
 <!DOCTYPE eagle SYSTEM "eagle.dtd">
-<eagle version="9.3.2">
+<eagle version="9.3.0">
 <drawing>
 <settings>
@@
 <layer number="25" name="tNames" color="7" fill="1" visible="yes" active="yes"/>
 <layer number="26" name="bNames" color="7" fill="1" visible="yes" active="yes"/>
-<layer number="27" name="tValues" color="7" fill="1" visible="no" active="yes"/>
+<layer number="27" name="tValues" color="7" fill="1" visible="yes" active="yes"/>
 <layer number="28" name="bValues" color="7" fill="1" visible="no" active="yes"/>
-<layer number="29" name="tStop" color="7" fill="3" visible="no" active="yes"/>
-<layer number="30" name="bStop" color="7" fill="6" visible="no" active="yes"/>
-<layer number="31" name="tCream" color="7" fill="4" visible="no" active="yes"/>
+<layer number="29" name="tStop" color="7" fill="3" visible="yes" active="yes"/>
+<layer number="30" name="bStop" color="7" fill="6" visible="yes" active="yes"/>
+<layer number="31" name="tCream" color="7" fill="4" visible="yes" active="yes"/>
 <layer number="32" name="bCream" color="7" fill="5" visible="no" active="yes"/>
 <layer number="33" name="tFinish" color="6" fill="3" visible="no" active="yes"/>
@@
 <layer number="42" name="bRestrict" color="1" fill="10" visible="yes" active="yes"/>
 <layer number="43" name="vRestrict" color="2" fill="10" visible="no" active="yes"/>
-<layer number="44" name="Drills" color="7" fill="1" visible="no" active="yes"/>
-<layer number="45" name="Holes" color="7" fill="1" visible="no" active="yes"/>
-<layer number="46" name="Milling" color="3" fill="1" visible="no" active="yes"/>
+<layer number="44" name="Drills" color="7" fill="1" visible="yes" active="yes"/>
+<layer number="45" name="Holes" color="7" fill="1" visible="yes" active="yes"/>
+<layer number="46" name="Milling" color="3" fill="1" visible="yes" active="yes"/>
 <layer number="47" name="Measures" color="7" fill="1" visible="no" active="yes"/>
 <layer number="48" name="Document" color="7" fill="1" visible="no" active="yes"/>
@@
 <layer number="119" name="KAP_TEKEN" color="7" fill="1" visible="no" active="yes"/>
 <layer number="120" name="Descript" color="7" fill="1" visible="no" active="yes"/>
-<layer number="121" name="_tsilk" color="7" fill="1" visible="no" active="yes"/>
+<layer number="121" name="_tPlace" color="14" fill="1" visible="yes" active="yes"/>
 <layer number="122" name="_bsilk" color="7" fill="1" visible="no" active="yes"/>
 <layer number="123" name="tTestmark" color="7" fill="1" visible="no" active="yes"/>
 <layer number="124" name="bTestmark" color="7" fill="1" visible="no" active="yes"/>
-<layer number="125" name="_tNames" color="7" fill="1" visible="no" active="yes"/>
+<layer number="125" name="_tNames" color="14" fill="1" visible="yes" active="yes"/>
 <layer number="126" name="_bNames" color="7" fill="1" visible="no" active="yes"/>
 <layer number="127" name="_tValues" color="7" fill="1" visible="no" active="yes"/>
@@
 <hole x="34" y="19.5" drill="3"/>
 <hole x="34" y="3" drill="3"/>
-<text x="19.05" y="1.905" size="1.778" layer="21" font="vector" ratio="12">the SPICE</text>
-<text x="36.83" y="1.905" size="0.8" layer="21" ratio="12">hv0a 1918</text>
+<text x="19.05" y="1.905" size="1.778" layer="21" font="vector" ratio="12">the SPIce</text>
+<text x="10.541" y="18.796" size="0.799996875" layer="125" font="vector" ratio="15" rot="R90" align="center">C1</text>
+<text x="17.399" y="17.7165" size="0.799996875" layer="125" font="vector" ratio="15" align="center">C2</text>
+<text x="11.43" y="5.334" size="0.799996875" layer="125" font="vector" ratio="15" align="center">C3</text>
+<text x="9.8425" y="5.334" size="0.799996875" layer="125" font="vector" ratio="15" align="center">C4</text>
+<text x="19.939" y="10.287" size="0.799996875" layer="125" font="vector" ratio="15" rot="R270" align="center">C5</text>
+<text x="19.05" y="17.7165" size="0.799996875" layer="125" font="vector" ratio="15" align="center">C6</text>
+<text x="23.8125" y="6.604" size="0.799996875" layer="125" font="vector" ratio="15" align="center">C7</text>
+<text x="35.7505" y="17.2085" size="0.799996875" layer="125" font="vector" ratio="15" rot="R180" align="center">C8</text>
+<text x="8.60300625" y="12.840996875" size="0.799996875" layer="121" font="vector" ratio="15">D1</text>
+<text x="8.509" y="1.143" size="0.799996875" layer="125" font="vector" ratio="15" align="center">D2</text>
+<text x="12.2555" y="1.143" size="0.799996875" layer="125" font="vector" ratio="15" rot="R180" align="center">D3</text>
+<text x="16.1925" y="1.143" size="0.799996875" layer="125" font="vector" ratio="15" rot="R180" align="center">D4</text>
+<text x="41.275" y="19.05" size="0.799996875" layer="125" font="vector" ratio="15" rot="R180" align="center">D5</text>
+<text x="7.62" y="17.2085" size="0.799996875" layer="125" font="vector" ratio="15" rot="R180" align="center">F1</text>
+<text x="45.8255125" y="11.697996875" size="0.799996875" layer="121" font="vector" ratio="15" rot="R270">J2</text>
+<text x="6.858" y="1.0795" size="0.799996875" layer="125" font="vector" ratio="15" rot="R180" align="center">R1</text>
+<text x="13.208" y="6.1595" size="0.799996875" layer="125" font="vector" ratio="15" align="center">R2</text>
+<text x="10.668" y="1.143" size="0.799996875" layer="125" font="vector" ratio="15" rot="R180" align="center">R3</text>
+<text x="14.605" y="1.143" size="0.799996875" layer="125" font="vector" ratio="15" rot="R180" align="center">R4</text>
+<text x="42.095496875" y="14.983509375" size="0.799996875" layer="125" font="vector" ratio="15" rot="R270" align="center">R5</text>
+<text x="42.158996875" y="9.983496875" size="0.799996875" layer="125" font="vector" ratio="15" rot="R90" align="center">R6</text>
+<text x="42.158996875" y="6.19000625" size="0.799996875" layer="125" font="vector" ratio="15" rot="R270" align="center">R7</text>
+<text x="13.2715" y="18.4785" size="0.799996875" layer="125" font="vector" ratio="15" rot="R90" align="center">U1</text>
+<text x="18.48" y="12.146509375" size="0.799996875" layer="121" font="vector" ratio="15" rot="R90">U2</text>
+<text x="13.6525" y="14.859" size="0.799996875" layer="121" font="vector" ratio="15" rot="R180">U3</text>
+<text x="28.448" y="8.328990625" size="0.799996875" layer="121" font="vector" ratio="15" rot="R270">U4</text>
+<text x="28.3845" y="10.702009375" size="0.799996875" layer="121" font="vector" ratio="15" rot="R270">U5</text>
+<text x="20.5105" y="13.39250625" size="0.799996875" layer="121" font="vector" ratio="15" rot="R270">U6</text>
+<text x="28.3845" y="13.39250625" size="0.799996875" layer="121" font="vector" ratio="15" rot="R270">U7</text>
+<text x="20.5105" y="15.8925" size="0.799996875" layer="121" font="vector" ratio="15" rot="R270">U8</text>
+<text x="28.3845" y="15.829" size="0.799996875" layer="121" font="vector" ratio="15" rot="R270">U9</text>
+<text x="17.5895" y="6.731" size="0.799996875" layer="121" font="vector" ratio="15">U10</text>
+<text x="31.158509375" y="7.222996875" size="0.799996875" layer="125" font="vector" ratio="15" align="center">U11</text>
+<text x="17.7165" y="14.859" size="0.799996875" layer="121" font="vector" ratio="15" rot="R180">U12</text>
+<text x="23.8125" y="17.7165" size="0.799996875" layer="121" font="vector" ratio="15" rot="R180">U13</text>
+<text x="27.6225" y="17.8435" size="0.799996875" layer="121" font="vector" ratio="15" rot="R180">U14</text>
+<text x="20.5105" y="11.210009375" size="0.799996875" layer="121" font="vector" ratio="15" rot="R270">U15</text>
+<text x="20.447" y="8.646490625" size="0.799996875" layer="121" font="vector" ratio="15" rot="R270">U16</text>
+<text x="7.112" y="7.439990625" size="0.799996875" layer="125" font="vector" ratio="15" rot="R90">USB1</text>
 </plain>
 <attributes>
@@
 <attribute name="VALUE" x="10.16" y="23.495" size="1.27" layer="27" rot="R180"/>
 </element>
-<element name="U$1" library="Utility &gt; Silkscreen" package="DESIGNEDINPT" value="" x="20.955" y="8.3185" smashed="yes" rot="MR0"/>
-<element name="U$3" library="Utility &gt; Silkscreen" package="RAFAEL_SILVA_5MM_ALT_3" value="" x="23.495" y="13.335" smashed="yes" rot="MR0"/>
-<element name="U$2" library="Utility &gt; Silkscreen" package="OSHW-LOGO-MINI" value="" x="30.7975" y="17.145" smashed="yes"/>
 <element name="USB1" library="Connectors &gt; USB" package="USB-MICRO-SMD" value="USB_MICRO-MICRO-B-SMT" x="2.032" y="11.25" smashed="yes">
 <attribute name="NAME" x="7.112" y="7.44" size="0.8" layer="25" font="vector" ratio="15" rot="R90"/>
 </element>
+<element name="U$1" library="Utility &gt; Silkscreen" package="DESIGNEDINPT" value="" x="17.155" y="1.7185" smashed="yes" rot="MR0"/>
+<element name="U$2" library="Utility &gt; Silkscreen" package="OSHW-LOGO-MINI" value="" x="31.0625" y="17.275" smashed="yes"/>
+<element name="U$4" library="Utility &gt; Silkscreen" package="RAFAEL_SILVA_10MM_ALT" value="" x="31.6" y="6.4" smashed="yes" rot="MR0"/>
 </elements>
 <signals>
